Commit message: updated

File: resources/robots/jet/urdf/jet.urdf (robot description, URDF)
Before this commit: robot dyros_jet_robot, 27 links, 26 joints
Joints:
- joint L_AnklePitch: limit lower=-1.57 upper=1.57 effort=800 velocity=20 -> lower=-1.57 upper=1.57 effort=1500 velocity=20
- joint L_HipPitch: limit lower=-3.14 upper=3.14 effort=1200 velocity=20 -> lower=-3.14 upper=3.14 effort=2000 velocity=20
- joint L_KneePitch: limit lower=0. upper=3. effort=1200 velocity=20 -> lower=0. upper=3. effort=2000 velocity=20
- joint R_AnklePitch: limit lower=-1.57 upper=1.57 effort=800 velocity=20 -> lower=-1.57 upper=1.57 effort=1200 velocity=20
- joint R_HipPitch: limit lower=-3.14 upper=3.14 effort=1200 velocity=20 -> lower=-3.14 upper=3.14 effort=2000 velocity=20
- joint R_KneePitch: limit lower=-3.14 upper=0. effort=1200 velocity=20 -> lower=-3.14 upper=0. effort=2000 velocity=20

Commit message: jet project finish

File: resources/robots/jet/urdf/jet.urdf (robot description, URDF)
Before this commit: robot dyros_jet_robot, 27 links, 26 joints
Joints:
- joint L_AnklePitch: limit lower=-1.57 upper=1.57 effort=1500 velocity=20 -> lower=-1.57 upper=1.57 effort=500 velocity=20
- joint L_HipPitch: limit lower=-3.14 upper=3.14 effort=2000 velocity=20 -> lower=-3.14 upper=3.14 effort=800 velocity=20
- joint L_HipYaw: limit lower=-1. upper=1. effort=100 velocity=20 -> lower=-1. upper=0. effort=100 velocity=20
- joint L_KneePitch: limit lower=0. upper=3. effort=2000 velocity=20 -> lower=0. upper=3. effort=800 velocity=20
- joint R_AnklePitch: limit lower=-1.57 upper=1.57 effort=1200 velocity=20 -> lower=-1.57 upper=1.57 effort=500 velocity=20
- joint R_HipPitch: limit lower=-3.14 upper=3.14 effort=2000 velocity=20 -> lower=-3.14 upper=3.14 effort=800 velocity=20
- joint R_HipYaw: limit lower=-1. upper=1. effort=100 velocity=20 -> lower=-0. upper=1. effort=100 velocity=20
- joint R_KneePitch: limit lower=-3.14 upper=0. effort=2000 velocity=20 -> lower=-3.14 upper=0. effort=800 velocity=20
- joint R_ShoulderPitch: limit lower=-0.0 upper=1.0 effort=300 velocity=100 -> lower=-1.0 upper=0.0 effort=300 velocity=100
- joint WaistYaw: limit lower=-1. upper=1.0 effort=300 velocity=100 -> lower=-1. upper=1.0 effort=100 velocity=20

File: resources/robots/jet/urdf/jet_fixed_centroid.urdf (robot description, URDF)
Before this commit: robot dyros_jet_robot, 16 links, 15 joints
Joints:
- joint WaistYaw: type fixed -> revolute
