Commit message: Asym Actor Critic updated

File: resources/robots/bolt10/urdf/bolt10.urdf (robot description, URDF)
Before this commit: robot bolt10_urdf, 11 links, 10 joints
Joints:
- joint L_AnklePitch_Joint: limit lower=-1.50 upper=1.50 effort=3.5 velocity=50 -> lower=-1.0 upper=1.50 effort=3.5 velocity=20
- joint L_HipPitch_Joint: limit lower=-1.57 upper=1.57 effort=4.4 velocity=50 -> lower=-1.57 upper=1.57 effort=4.4 velocity=20
- joint L_HipRoll_Joint: limit lower=-0.73 upper=1.57 effort=3.5 velocity=50 -> lower=-0.73 upper=1.57 effort=3.5 velocity=20
- joint L_HipYaw_Joint: limit lower=-0.43 upper=1.57 effort=3.5 velocity=50 -> lower=-0.43 upper=1.57 effort=3.5 velocity=20
- joint L_KneePitch_Joint: limit lower=0 upper=3.14 effort=4.4 velocity=50 -> lower=0 upper=3.14 effort=4.4 velocity=20
- joint R_AnklePitch_Joint: limit lower=-1.50 upper=1.50 effort=3.5 velocity=50 -> lower=-1.0 upper=1.50 effort=3.5 velocity=20
- joint R_HipPitch_Joint: limit lower=-1.57 upper=1.57 effort=4.4 velocity=50 -> lower=-1.57 upper=1.57 effort=4.4 velocity=20
- joint R_HipRoll_Joint: limit lower=-1.57 upper=0.73 effort=3.5 velocity=50 -> lower=-1.57 upper=0.73 effort=3.5 velocity=20
- joint R_HipYaw_Joint: limit lower=-1.57 upper=0.43 effort=3.5 velocity=50 -> lower=-1.57 upper=0.43 effort=3.5 velocity=20
- joint R_KneePitch_Joint: limit lower=0 upper=3.14 effort=4.4 velocity=50 -> lower=0 upper=3.14 effort=4.4 velocity=20

Commit message: ICRA workshop

File: resources/robots/bolt10/urdf/bolt10.urdf (robot description, URDF)
Before this commit: robot bolt10_urdf, 11 links, 10 joints
Links:
- link L_Foot: geometry collision box size=0.10 0.03 0.02; visual mesh filename=../meshes/L_Foot.stl
- link R_Foot: geometry collision box size=0.10 0.03 0.02; visual mesh filename=../meshes/R_Foot.stl
Joints:
- joint L_AnklePitch_Joint: limit lower=-1.0 upper=1.50 effort=3.5 velocity=20 -> lower=-1.0 upper=1.50 effort=3.5 velocity=5
- joint R_AnklePitch_Joint: limit lower=-1.0 upper=1.50 effort=3.5 velocity=20 -> lower=-1.0 upper=1.50 effort=3.5 velocity=5
