Commit message: Deep mimic updated

File: resources/robots/cassie/urdf/cassie.urdf (robot description, URDF)
Before this commit: robot cassie, 16 links, 15 joints
Joints:
- joint ankle_joint_left: limit lower=0.6458 upper=2.8623 effort=195 velocity=20.5085 -> lower=0.6458 upper=2.8623 effort=195 velocity=5
- joint ankle_joint_right: limit lower=0.6458 upper=2.8623 effort=195 velocity=20.5085 -> lower=0.6458 upper=2.8623 effort=195 velocity=5
- joint hip_abduction_left: limit lower=-0.2618 upper=0.3927 effort=112 velocity=20.1475 -> lower=-0.2618 upper=0.3927 effort=112 velocity=5
- joint hip_abduction_right: limit lower=-0.3927 upper=0.2618 effort=112 velocity=20.1475 -> lower=-0.3927 upper=0.2618 effort=112 velocity=5
- joint hip_flexion_left: limit lower=-0.8727 upper=1.3963 effort=195 velocity=20.5085 -> lower=-0.8727 upper=1.3963 effort=195 velocity=5
- joint hip_flexion_right: limit lower=-0.8727 upper=1.3963 effort=195 velocity=20.5085 -> lower=-0.8727 upper=1.3963 effort=195 velocity=5
- joint hip_rotation_left: limit lower=-0.3927 upper=0.3927 effort=112 velocity=20.1475 -> lower=-0.3927 upper=0.3927 effort=112 velocity=5
- joint hip_rotation_right: limit lower=-0.3927 upper=0.3927 effort=112 velocity=20.1475 -> lower=-0.3927 upper=0.3927 effort=112 velocity=5
- joint thigh_joint_left: limit lower=-2.8623 upper=-0.6458 effort=195 velocity=20.5085 -> lower=-2.8623 upper=-0.6458 effort=195 velocity=5
- joint thigh_joint_right: limit lower=-2.8623 upper=-0.6458 effort=195 velocity=20.5085 -> lower=-2.8623 upper=-0.6458 effort=195 velocity=5
- joint toe_joint_left: limit lower=-2.4435 upper=-0.5236 effort=45 velocity=20.5192 -> lower=-2.4435 upper=-0.5236 effort=45 velocity=5
- joint toe_joint_right: limit lower=-2.4435 upper=-0.5236 effort=45 velocity=20.5192 -> lower=-2.4435 upper=-0.5236 effort=45 velocity=5
